Commit message: Finish tuning my_bot parameters

File: my_bot/urdf/material.xacro (robot description, xacro)
@@ -1,4 +1,4 @@
-<? xml version="1.0" ?>
-<robot name="my_bot" xmlns:xacro="https://www.ros.org/wiki/xacro" >
+<?xml version='1.0'?>
+<robot name="my_bot" xmlns:xacro="http://www.ros.org/wiki/xacro">
 <material name="black">
 <color rgba="0.0 0.0 0.0 1.0" />
@@ -10,5 +10,5 @@
 <color rgba="0.0 0.8 0.0 1.0" />
 </material>
-<material name="blue">
+<material name="red">
 <color rgba="0.8 0.0 0.0 1.0" />
 </material>

File: my_bot/urdf/my_bot.xacro (robot description, xacro)
@@ -74,5 +74,5 @@
         <cylinder radius="0.1" length="0.05"/>
       </geometry>
-      </material name="black">
+      <material name="black"/>
     </visual>
      <collision name='front_right_wheel_collision'>
@@ -101,5 +101,5 @@
   </joint>
    <!-- back  left wheel model -->
-  <link name="backt_left_wheel">
+  <link name="back_left_wheel">
   	 <visual name='back_left_wheel_visual'>
       <origin xyz="0 0 0" rpy=" 0 1.5707 1.5707"/>
@@ -140,5 +140,5 @@
         <cylinder radius="0.1" length="0.05"/>
       </geometry>
-      </material name="black">
+      <material name="black"/>
     </visual>
      <collision name='back_right_wheel_collision'>
@@ -200,5 +200,5 @@
       <origin xyz="0 0 0" rpy=" 0 0 0"/>
       <geometry>
-        <mesh filename="package://udacity_bot/meshes/hokuyo.dae"/>
+        <mesh filename="package://my_bot/meshes/hokuyo.dae"/>
       </geometry>
     </visual>
@@ -223,4 +223,5 @@
     <parent link="chassis" />
     <child link="hokuyo" />
+    <axis xyz="1 0 0" rpy="0 0 0"/>
   </joint>
 </robot>

File: udacity_bot/urdf/udacity_bot.xacro (robot description, xacro)
@@ -177,4 +177,5 @@
     <parent link="chassis" />
     <child link="hokuyo" />
+    <axis xyz="1 0 0" rpy="0 0 0"/>
   </joint>
 </robot>
